File: eval/eval.kicad_sch (KiCad schematic)
At the start: 5 parts, among them J1 TC2030, U9 STM32G0B1CBTx

Commit message: [layout] first draft layout
Other:
- sheet power_mux renamed power_mux(page 10)
- sheet power_battery ports: added FROM_BUCK, I_OUT_MON, TO_BATT, ~{fault_reset_mcu}; removed none
- note added: "Peripheral"
- note added: "Power path"

Commit message: [layout] 50*100mm, without trace
Other:
- sheet power_mux(page 10) renamed power_mux
- sheet power_usb_pd (page 9) renamed power_usb_pd
- added sheet power_dc_in (power_dc_in.kicad_sch)
Changed lines of the file:
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@@
+	(wire
+		(pts
+			(xy 198.12 78.74) (xy 208.28 78.74)
+		)
+		(stroke
+			(width 0.5)
+			(type default)
+		)
+	)
 	(wire
 		(pts
@@
 	(wire
 		(pts
+			(xy 208.28 57.15) (xy 215.9 57.15)
+		)
+		(stroke
+			(width 0.5)
+			(type default)
+		)
+	)
+	(wire
+		(pts
 			(xy 68.58 157.48) (xy 68.58 154.94)
 		)
@@
 		(stroke
 			(width 0)
+			(type default)
+		)
+	)
+	(wire
+		(pts
+			(xy 208.28 78.74) (xy 208.28 57.15)
+		)
+		(stroke
+			(width 0.5)
 			(type default)
 		)
@@
 			(project "eval"
 				(path "/8b023652-20db-48ce-ad53-bc2d9a4e5dd4"
-					(page "2")
+					(page "10")
 				)
 			)
@@
 			(project "eval"
 				(path "/8b023652-20db-48ce-ad53-bc2d9a4e5dd4"
-					(page "8")
+					(page "14")
 				)
 			)
@@
 			(color 0 0 0 0)
 		)
-		(property "Sheetname" "power_usb_pd (page 9)"
+		(property "Sheetname" "power_usb_pd"
 			(at 175.26 46.2784 0)
 			(show_name no)
@@
 			(project "eval"
 				(path "/8b023652-20db-48ce-ad53-bc2d9a4e5dd4"
-					(page "9")
+					(page "12")
+				)
+			)
+		)
+	)
+	(sheet
+		(at 175.26 73.66)
+		(size 22.86 10.34)
+		(exclude_from_sim no)
+		(in_bom yes)
+		(on_board yes)
+		(dnp no)
+		(fields_autoplaced yes)
+		(stroke
+			(width 0.1524)
+			(type solid)
+		)
+		(fill
+			(color 0 0 0 0)
+		)
+		(property "Sheetname" "power_dc_in"
+			(at 175.26 72.9484 0)
+			(show_name no)
+			(do_not_autoplace no)
+			(effects
+				(font
+					(size 1.27 1.27)
+				)
+				(justify left bottom)
+			)
+		)
+		(property "Sheetfile" "power_dc_in.kicad_sch"
+			(at 175.26 84.5846 0)
+			(show_name no)
+			(do_not_autoplace no)
+			(effects
+				(font
+					(size 1.27 1.27)
+				)
+				(justify left top)
+			)
+		)
+		(pin "VDC" output
+			(at 198.12 78.74 0)
+			(effects
+				(font
+					(size 1.27 1.27)
+				)
+				(justify right)
+			)
+		)
+		(instances
+			(project "eval"
+				(path "/8b023652-20db-48ce-ad53-bc2d9a4e5dd4"
+					(page "13")
 				)
 			)
@@
 			(color 0 0 0 0)
 		)
-		(property "Sheetname" "power_mux(page 10)"
+		(property "Sheetname" "power_mux"
 			(at 215.9 44.1384 0)
 			(show_name no)
@@
 			(project "eval"
 				(path "/8b023652-20db-48ce-ad53-bc2d9a4e5dd4"
-					(page "10")
-				)
-			)
+					(page "11")
+				)
+			)
