File: eval/power_battery.kicad_sch (KiCad schematic)
At the start: 36 parts, among them Q9 2N7002, U17 HYG015N03LS1C2, U18 MX74502D23_C41433189, U19 TLV3501AIDBV, U21 HYG015N03LS1C2, U22 74LVC1G32, U5 TLV3501AIDBV

Commit message: [sim] verity TLV3501 with RC output
Parts:
- removed U22: 74LVC1G32, symbol 74xGxx:74LVC1G32
- added D6: BAV70, Package_TO_SOT_SMD:SOT-23, symbol Diode:BAV70
- added R68: 1M, Resistor_SMD:R_0603_1608Metric, symbol Device:R_Small
- R55, R56: value 100 -> 2.2
Connections:
- net +3V3: no longer C60.2
- net GNDA: now also R68.2
- net NEG_V: now also D6.1 (A)
- net OV: now also C60.2, D6.3 (K), R68.1
- net OVER_I: now also D6.2 (A)
Other:
- note removed: "TODO: 1. design feedback block to latch error state 2. route push-pull output to gpio to detect error 1. remove latch 2. let mcu latch"
- moved on the sheet: C49, C50, C51, C55, C56, C57, C58, C59, C61, Q9, R46, R49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

Commit message: [sch] Remove RC delay, add 74lvc trigger
Parts:
- removed C60: 100n, Capacitor_SMD:C_0603_1608Metric, symbol Device:C_Small
- removed R55, R56: 2.2, Resistor_SMD:R_0603_1608Metric, symbol Device:R_Small
- removed R68: 1M, Resistor_SMD:R_0603_1608Metric, symbol Device:R_Small
- added C13: 22p, symbol Device:C_Small
- added C17: 1u, symbol Device:C_Small
- added R25: 33k, symbol Device:R_Small
- added R44: 10, symbol Device:R_Small
- added R45: 200k, symbol Device:R_Small
- added U20: SN74LVC1G123DCUR_C352969, EasyEDA:VSSOP-8_L2.3-W2.0-P0.50-LS3.1-BL, symbol EasyEDA:SN74LVC1G123DCUR_C352969
Connections:
- net +3V3: now also R45.1, U20.3 (~{CLR}), U20.8 (VCC)
- net GNDA: now also C13.2, R25.2, U20.1 (~{A}), U20.4 (GND)
- net NEG_V: now also R61.2, TP7.1, U5.5
- net OV: now also U20.5 (Q); no longer D6.3 (K)
- net OVER_I: now also R62.2, TP8.1, U19.5
- new net: C17.1, R45.2, U20.7 (Rext/Cext)
- new net: C17.2, U20.6 (Cext)
- new net: C13.1, R25.1, R44.2, U20.2 (B)
- new net: D6.3 (K), R44.1
Other:
- note added: "5Hz Hiccup"
- moved on the sheet: C50, Q9, R46, TP3
