File: eval/power_battery.kicad_sch (KiCad schematic)
At the start: 40 parts, among them Q9 2N7002, U17 HYG015N03LS1C2, U18 MX74502D23_C41433189, U19 TLV3501AIDBV, U20 SN74LVC1G123DCUR_C352969, U21 HYG015N03LS1C2, U5 TLV3501AIDBV

Commit message: [layout&trace] layout 3 ntc sense.
Need more trace for 3 ntc, need add filter capacitor
Connections:
- net VBATT is gone; now on net TO_BATT: R49.1
Changed lines of the file:
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@@
+	(hierarchical_label "TO_BATT"
+		(shape input)
+		(at 167.64 35.56 180)
+		(effects
+			(font
+				(size 1.27 1.27)
+			)
+			(justify right)
+		)
+	)
 	(hierarchical_label "TO_BATT"
 		(shape input)
@@
 		)
 	)
-	(hierarchical_label "VBATT"
-		(shape input)
-		(at 167.64 35.56 180)
-		(effects
-			(font
-				(size 1.27 1.27)
-			)
-			(justify right)
-		)
-	)
