File: eval/eval.kicad_pcb (KiCad board)
At the start: 4 copper layers, 49.2 x 98 mm, 186 parts, among them CN1 XT30PW-M, J1 TC2030, Q1 DMG2302UK-7, Q10 2N7002, Q2 BSC0702LS, Q3 BSC0702LS, Q4 BSC0702LS, Q5 BSC0702LS, Q6 WSD4070DN, Q7 WSD4070DN, Q8 AP40P04Q, Q9 2N7002, U1 STM32G0B1CBTx, U10 INA180A3, U11 INA180A3, U12 MX74700T_C22468156, U13 MX74700T_C22468156, U14 RCLAMP0521T-ES, U15 RCLAMP0521T-ES, U16 HUSB238A-BB001-QN16R, U17 HYG015N03LS1C2, U18 MX74502D23_C41433189, U19 SN74LVC1G00DBV, U2 TLV9062, U20 SN74LVC1G00DBV, U21 HYG015N03LS1C2, U22 LM2903, U23 TLV3501AIDBV, U24 TS34031, U25 TS34031, U3 TPS7A2033PDBVR, U4 AP63205WU-7, U6 HS096T01H13, U7 TLV9061xDBV, U8 TCAN1044VDRBRQ1, U9 LM5148RGYR

Commit message: [layout] change latch -> trigger& software latch (plan)
Parts:
- removed C52, C62, C63: 100n, Capacitor_SMD:C_0603_1608Metric
- removed C53: 1u, Capacitor_SMD:C_0603_1608Metric
- removed C54: 10n, Capacitor_SMD:C_0603_1608Metric
- removed JP1, JP2, JP3, JP4: SolderJumper_2_Bridged, Jumper:SolderJumper-2_P1.3mm_Bridged_RoundedPad1.0x1.5mm
- removed Q10: 2N7002, Package_TO_SOT_SMD:SOT-23
- removed R48: 100, Resistor_SMD:R_0603_1608Metric
- removed R50: 22k, Resistor_SMD:R_0603_1608Metric
- removed R51: 15k, Resistor_SMD:R_0603_1608Metric
- removed R55, R56: 10k, Resistor_SMD:R_0603_1608Metric
- removed TP1: 74502_ov, TestPoint:TestPoint_Pad_D2.0mm
- removed TP2: fault_reset_mcu, TestPoint:TestPoint_Pad_D2.0mm
- removed TP3: power_on_hold_rc, TestPoint:TestPoint_Pad_D2.0mm
- removed TP4: 74502_en, TestPoint:TestPoint_Pad_D2.0mm
- removed TP5: fault_latch, TestPoint:TestPoint_Pad_D2.0mm
- removed TP6: drop_volt, TestPoint:TestPoint_Pad_D2.0mm
- removed U22: LM2903, Package_SO:TSSOP-8_4.4x3mm_P0.65mm
- removed U23: TLV3501AIDBV, Package_TO_SOT_SMD:SOT-23-6
- added C13: 22p, Capacitor_SMD:C_0603_1608Metric, F.Cu at (72.1, 139.5)
- added C17: 1u, Capacitor_SMD:C_0603_1608Metric, F.Cu at (64.3, 139.4)
- added C21: 470u@35v, Capacitor_SMD:C_0603_1608Metric, F.Cu at (100.3, 144.8)
- added R25: 33k, Resistor_SMD:R_0603_1608Metric, F.Cu at (70.6, 139.4)
- added R63: R, Resistor_SMD:R_0603_1608Metric, F.Cu at (118.3, 144.8)
- added R64: R, Resistor_SMD:R_0603_1608Metric, F.Cu at (112.3, 144.8)
- added R65: R, Resistor_SMD:R_0603_1608Metric, F.Cu at (106.3, 144.8)
- added R69: 1k, Resistor_SMD:R_0603_1608Metric, F.Cu at (108.3, 135.2)
- added R70: 100k, Resistor_SMD:R_0603_1608Metric, F.Cu at (108.3, 137.7)
- added TH1: Thermistor_NTC, Resistor_SMD:R_0603_1608Metric, F.Cu at (118.3, 147.3)
- added TH2: Thermistor_NTC, Resistor_SMD:R_0603_1608Metric, F.Cu at (112.3, 147.3)
- added TH3: Thermistor_NTC, Resistor_SMD:R_0603_1608Metric, F.Cu at (106.3, 147.3)
- added U5: TLV3501AIDBV, Package_TO_SOT_SMD:SOT-23-6, F.Cu at (68.7, 147.6)
- C56: value 4.7n -> 100p
- C57: value 1n -> 100n
- C58: value 100n -> 1n
- C60: value 1u -> 100n
- C61: value 47n -> 1n
- D6: value BAT54J -> BAV70; footprint Diode_SMD:D_SOD-323F -> Package_TO_SOT_SMD:SOT-23
- R44: value 1k -> 10
- R45: value 1k -> 200k
- R54: value 4.7k -> 10k
- R59: value 8.06k -> 13K
- R60: value 24.9k -> 24.3K
- R62: value 500k -> 100
- TP7, TP8: moved to F.Cu
- U19: value SN74LVC1G00DBV -> TLV3501AIDBV; footprint Package_TO_SOT_SMD:SOT-23-5 -> Package_TO_SOT_SMD:SOT-23-6
- U20: value SN74LVC1G00DBV -> SN74LVC1G123DCUR_C352969; footprint Package_TO_SOT_SMD:SOT-23-5 -> EasyEDA:VSSOP-8_L2.3-W2.0-P0.50-LS3.1-BL
- moved TP7 122.5 mm to (151.4, 141.5), turned to 0 degrees
- moved TP8 122.5 mm to (151.4, 145.5), turned to 0 degrees
- moved R25 46.8 mm to (94.3, 64.8)
- moved H4 36.8 mm to (59.1, 163.7)
- moved C59 19.7 mm to (77.7, 150.4)
- moved R62 14.9 mm to (78.3, 145.0), turned to 0 degrees
- moved D6 14.8 mm to (76.5, 140.2), turned to 90 degrees
- moved C57 13.2 mm to (68.6, 150.4), turned to 0 degrees
- moved C61 12.9 mm to (74.9, 146.6)
- moved U20 12.2 mm to (67.3, 139.2)
- moved C60 11.9 mm to (68.1, 141.7), turned to 180 degrees
- moved R44 11.8 mm to (73.7, 139.4), turned to -90 degrees
- moved R45 9.97 mm to (65.0, 141.7), turned to 180 degrees
- moved C50 9.88 mm to (55.1, 142.3)
- moved R46 9.88 mm to (53.6, 142.3)
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Connections:
- net /power_battery/GATE renamed /power_battery_protection/GATE
- net /power_battery/VBATT renamed /power_battery_protection/VBATT
- net /power_battery/vbat_comp_thre renamed /power_battery_protection/vbat_comp_thre
- net /power_battery/vbat_none_neg renamed /power_battery_protection/vbat_none_neg
- C56 pad 1: /power_battery/i_mon_filter -> Net-(U19-+)
- C57 pad 1: /power_battery/v_drop_fast -> GNDA
- C57 pad 2: GNDA -> +3V3
- C60 pad 1: +3V3 -> GNDA
- C60 pad 2: GNDA -> +3V3
- C61 pad 1: Net-(D6-K) -> GNDA
- C61 pad 2: GNDA -> /power_battery_protection/2V_REF
- D6 pad 1: Net-(D6-K) -> /power_battery_protection/NEG_V
- D6 pad 2: Net-(D6-A) -> /power_battery_protection/OVER_I
- Q9 pad 3: /power_battery/power_on_hold -> /power_battery_protection/EN
- R44 pad 1: +3V3 -> Net-(D6-K)
- R44 pad 2: /power_battery/power_on_hold -> Net-(U20-B)
- R45 pad 2: /power_battery/~{fault_reset_mcu} -> Net-(U20-Rext/Cext)
- R54 pad 2: /power_battery/i_mon_filter -> Net-(U19-+)
- R59 pad 2: /power_battery/2v5 -> /power_battery_protection/2V_REF
- R60 pad 1: /power_battery/2v5 -> /power_battery_protection/2V_REF
- R61 pad 1: Net-(R61-Pad1) -> /power_battery_protection/NEG_V_ALARM
- R61 pad 2: Net-(D6-A) -> /power_battery_protection/NEG_V
- R62 pad 1: Net-(D6-K) -> /power_battery_protection/OVER_I_ALARM
- R62 pad 2: GNDA -> /power_battery_protection/OVER_I
- TP7 pad 1: Net-(JP2-A) -> /power_battery_protection/NEG_V
- TP8 pad 1: Net-(JP3-A) -> /power_battery_protection/OVER_I
- U10 pad 1: Net-(R25-Pad1) -> /ADC_I_OUT_MON
- U18 pad 5: /power_battery/power_on_hold -> /power_battery_protection/EN
- U18 pad 7: /power_battery/OV -> /power_battery_protection/OV
- U19 pad 1: /power_battery/power_on_hold -> /power_battery_protection/2V_REF
- U19 pad 2: Net-(U19-Pad2) -> GNDA
- U19 pad 3: GNDA -> Net-(U19-+)
- U19 pad 4: /power_battery/fault_latch -> +3V3
- U19 pad 5: +3V3 -> /power_battery_protection/OVER_I
- U20 pad 1: /power_battery/fault_latch -> GNDA
- U20 pad 2: /power_battery/~{fault_reset_mcu} -> Net-(U20-B)
- U20 pad 3: GNDA -> +3V3
- U20 pad 4: Net-(U19-Pad2) -> GNDA
- U20 pad 5: +3V3 -> /power_battery_protection/OV
Routing:
- net +3V3: track 31.6 -> 18.6 mm, vias 9 -> 6
- net /power_battery/fault_latch: track 9.01 -> 0.00 mm
- net /power_battery_protection/vbat_none_neg: track 6.93 -> 0.00 mm
- net /power_battery/v_drop_slow: track 5.84 -> 0.00 mm
- net /power_battery_protection/vbat_comp_thre: track 5.69 -> 0.00 mm
- net /power_battery/v_drop_fast: track 5.58 -> 0.00 mm
- net /power_battery/2v5: track 4.81 -> 0.00 mm
- net /power_battery/i_mon_filter: track 4.11 -> 0.00 mm
- net /power_battery/~{fault_reset_mcu}: track 4.09 -> 0.00 mm
- net /power_battery/power_on_hold: track 6.40 -> 2.35 mm
- net Net-(U19-Pad2): track 4.05 -> 0.00 mm
- net Net-(Q9-G): track 5.43 -> 1.57 mm
- net Net-(R61-Pad1): track 3.51 -> 0.00 mm
- net Net-(D6-K): track 3.49 -> 0.00 mm
- net Net-(Q10-G): track 1.98 -> 0.00 mm
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
Commit message: [layout&trace] layout 3 ntc sense.
Need more trace for 3 ntc, need add filter capacitor
Parts:
- removed H5: 2.54-2*5P, EasyEDA:HDR-SMD_10P-P2.54-V-F-R2-C5-S2.54-LS7.4
- removed the R25 at (94.3, 64.8)
- removed R47: 1k, Resistor_SMD:R_0603_1608Metric
- removed R63: R, Resistor_SMD:R_0603_1608Metric
- removed TH1, TH2, TH3: Thermistor_NTC, Resistor_SMD:R_0603_1608Metric
- added C34: 100n, Capacitor_SMD:C_0603_1608Metric, F.Cu at (59.3, 91.2)
- added C52: 10n, Capacitor_SMD:C_0603_1608Metric, F.Cu at (61.0, 91.2)
- added C53: 100n, Capacitor_SMD:C_0603_1608Metric, F.Cu at (17.5, 94.5)
- added C54: 100n, Capacitor_SMD:C_0603_1608Metric, F.Cu at (14.8, 101.0)
- added C62: 100n, Capacitor_SMD:C_0603_1608Metric, F.Cu at (28.9, 113.3)
- added R50: 20k 0.1%, Resistor_SMD:R_0603_1608Metric, F.Cu at (53.4, 90.7)
- added R51: 10k 0.1%, Resistor_SMD:R_0603_1608Metric, F.Cu at (56.6, 92.5)
- added R55: 10k 0.1%, Resistor_SMD:R_0603_1608Metric, F.Cu at (56.6, 86.6)
- added R56: 100, Resistor_SMD:R_0603_1608Metric, F.Cu at (60.1, 88.5)
- added R68: 0, Resistor_SMD:R_0603_1608Metric, F.Cu at (38.1, 139.8)
- added R71: 0, Resistor_SMD:R_0603_1608Metric, F.Cu at (43.4, 69.6)
- added R72: R_Small, Resistor_SMD:R_0603_1608Metric, F.Cu at (63.8, 101.3)
- added R73: R_Small, Resistor_SMD:R_0603_1608Metric, F.Cu at (62.2, 101.3)
- added R74: 10k, Resistor_SMD:R_0603_1608Metric, F.Cu at (65.8, 101.3)
- added TH0: NTC_10k, Resistor_SMD:R_0603_1608Metric, F.Cu at (62.7, 112.2)
- added TP1: 74502_ov, TestPoint:TestPoint_Pad_D2.0mm, F.Cu at (94.7, 154.9)
- added TP10: TestPoint, TestPoint:TestPoint_Keystone_5015_Micro_Mini, F.Cu at (54.9, 101.9)
- added TP2: TestPoint, TestPoint:TestPoint_Keystone_5019_Miniature, F.Cu at (38.2, 135.1)
- added TP3: power_on_hold_rc, TestPoint:TestPoint_Pad_D2.0mm, F.Cu at (94.7, 159.0)
- added TP4: TestPoint, TestPoint:TestPoint_Keystone_5019_Miniature, F.Cu at (46.1, 71.0)
- added TP9: TestPoint, TestPoint:TestPoint_Keystone_5015_Micro_Mini, F.Cu at (54.9, 99.9)
- added U22: KH-1.27FH-2X10P-H4.3-SMT, EasyEDA:CONN-SMD_20P-P1.27_KINGHELM_KH-1.27FH-2X10P-H4.3-SMT, F.Cu at (72.9, 107.9)
- added U23: OPA333xxDBV, Package_TO_SOT_SMD:SOT-23-5, F.Cu at (56.7, 89.5)
- R13: value 10k -> 20k 0.1%
- R64, R65: value R -> 10k
- moved C18 246.7 mm to (102.9, 98.7), turned to -90 degrees
- moved R8 244.4 mm to (104.4, 98.7), turned to -90 degrees
- moved R9 243.0 mm to (102.9, 101.8), turned to -90 degrees
- moved Q1 236.4 mm to (106.8, 99.9), turned to 180 degrees
- moved C20 231.1 mm to (96.7, 98.9), turned to -90 degrees
- moved U7 222.0 mm to (99.6, 100.4)
- moved R12 221.2 mm to (95.1, 98.9)
- moved C19 213.7 mm to (95.1, 102.0), turned to -90 degrees
- moved R11 211.2 mm to (96.7, 102.0), turned to -90 degrees
- moved R10 203.1 mm to (93.6, 102.0), turned to 90 degrees
- moved C21 88.3 mm to (23.5, 101.3)
- moved R64 67.8 mm to (59.4, 102.4), turned to 180 degrees
- moved C37 66.0 mm to (23.5, 103.8)
- moved R65 64.2 mm to (59.4, 100.8), turned to 180 degrees
- moved R69 51.6 mm to (57.9, 146.1), turned to 180 degrees
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Connections:
- C1 pad 2: Net-(U1-VREF+) -> VREF
- C19 pad 1: /LCD_I_CTL -> Net-(U7-+)
- F2 pad 1: /power_buck/OUT_ISNS+ -> /VBAT-
- F2 pad 2: Net-(F2-Pad2) -> /power_buck/OUT_ISNS+
- F3 pad 1: /power_buck/OUT_ISNS+ -> /VBAT-
- F3 pad 2: Net-(F2-Pad2) -> /power_buck/OUT_ISNS+
- R10 pad 1: +3V3 -> /LCD_I_CTL
- R10 pad 2: /LCD_I_CTL -> Net-(U7-+)
- R11 pad 1: /LCD_I_CTL -> Net-(U7-+)
- R13 pad 1: GNDA -> /remote_sense/DIFF+
- R13 pad 2: /can/CAN_STB -> Net-(U23-+)
- R49 pad 1: /power_battery_protection/VBATT -> VBAT
- R61 pad 1: /power_battery_protection/NEG_V_ALARM -> /NEG_V_ALARM
- R62 pad 1: /power_battery_protection/OVER_I_ALARM -> /OVER_I_ALARM
- R64 pad 1: +2V5 -> VREF
- R64 pad 2: /ntc1/NTC_OUT -> /ADC_NTC_0
- R65 pad 1: +2V5 -> VREF
- R65 pad 2: /ntc2/NTC_OUT -> /ADC_NTC_1
- R69 pad 2: /power_battery_protection/MCU_EN -> /EN_OUTPUT_MOS
- U1 pad 10: /RST -> /~{RST}
- U1 pad 18: unconnected-(U1-PA7-Pad18) -> /ADC_I_OUT_MON
- U1 pad 19: /ADC_I_OUT_MON -> /ADC_V_OUT+_MON
- U1 pad 20: /ADC_V_OUT+_MON -> /ADC_V_OUT-_MON
- U1 pad 21: /ADC_V_OUT-_MON -> /ADC_NTC_2
- U1 pad 28: /BUCK_SYNC -> /KEY_1
- U1 pad 29: /UART1_TX -> /KEY_2
- U1 pad 30: unconnected-(U1-PC6-Pad30) -> /KEY_0
- U1 pad 32: /UART1_RX -> /KEY_3
- U1 pad 37: unconnected-(U1-PA15-Pad37) -> /RESERVED_1
- U1 pad 38: unconnected-(U1-PD0-Pad38) -> /RESERVED_0
- U1 pad 39: unconnected-(U1-PD1-Pad39) -> /OVER_I_ALARM
- U1 pad 40: unconnected-(U1-PD2-Pad40) -> /NEG_V_ALARM
- U1 pad 41: unconnected-(U1-PD3-Pad41) -> /EN_OUTPUT_MOS
- U1 pad 45: unconnected-(U1-PB6-Pad45) -> /UART1_TX
- U1 pad 46: /CAN_STB -> /UART1_RX
- U1 pad 5: Net-(U1-VREF+) -> VREF
- U25 pad 1: Net-(F2-Pad2) -> /VBAT-
- U25 pad 2: Net-(F2-Pad2) -> /VBAT-
- U25 pad 3: Net-(F2-Pad2) -> /VBAT-
- U25 pad 4: Net-(F2-Pad2) -> /VBAT-
- U7 pad 3: /LCD_I_CTL -> Net-(U7-+)
- U8 pad 8: /can/CAN_STB -> GNDA
Routing:
- net /OVER_I_ALARM: track 0.00 -> 94.6 mm, vias 0 -> 2
- net /NEG_V_ALARM: track 0.00 -> 87.1 mm, vias 0 -> 2
- net /EN_OUTPUT_MOS: track 0.00 -> 85.8 mm, vias 0 -> 2
- net /ADC_I_OUT_MON: track 11.6 -> 90.5 mm, vias 0 -> 2
- net /power_buck/VOUT: track 6.41 -> 79.8 mm, vias 0 -> 3
- net /DAC_I_SET: track 3.08 -> 69.9 mm
- net /DAC_V_SET: track 3.14 -> 68.7 mm
- net /remote_sense/DIFF+: track 0.00 -> 64.3 mm, vias 0 -> 10
- net /BUCK_EN: track 3.17 -> 45.5 mm, vias 0 -> 2
- net VREF: track 0.00 -> 35.0 mm, vias 0 -> 4
- net /remote_sense/DIFF-: track 0.00 -> 26.0 mm, vias 0 -> 10
- net /LCD_RST: track 0.00 -> 17.8 mm
- net Net-(U16-GATE): track 0.00 -> 17.3 mm
- net VBAT: track 0.00 -> 17.2 mm
- net /RESERVED_1: track 0.00 -> 16.0 mm, vias 0 -> 2
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