File: eval/power.kicad_sch (KiCad schematic)
At the start: 48 parts, among them Q1 BSC0702LS, Q2 BSC0702LS, Q5 BSC0702LS, Q6 BSC0702LS, U2 LM5148RGYR, U3 INA180A3, U8 INA180A3

Commit message: [layout] fan on bottom side, power area on top
Connections:
- net GNDPWR: now also R14.1, R46.1
- net V_OUT: now also C35.1, C40.1, C41.1, C42.1, C43.1, L1.1, R45.2, U2.21 (VOUT); no longer R14.1, R46.2
- removed net OUT_ISNS+: C35.1, C40.1, C41.1, C42.1, C43.1, L1.1, R13.1, R45.2, R46.1, U2.21 (VOUT)
- new net GNDPWR_BAT: R13.1, R46.2

Commit message: [trace] add high power trace
Parts:
- added R66, R67: R_Small, Resistor_SMD:R_0603_1608Metric, symbol Device:R_Small
- renumbered C34 to C21, C8 to C22, C9 to C23, C36 to C24, C37 to C25, C7 to C26, C12 to C27, C17 to C28, C2 to C29, C33 to C30, C1 to C31, C6 to C32, C25 to C33, C10 to C34, C18 to C35, C4 to C36, C45 to C37, C46 to C38, C5 to C39, C39 to C40, C40 to C41, C41 to C42, C42 to C43, C43 to C44, C35 to C45, L1 to L2, Q6 to Q2, Q1 to Q3, Q5 to Q4, Q2 to Q5, R1 to R14, R2 to R15, R4 to R16, R5 to R17, R3 to R18, R13 to R19, R14 to R20, R6 to R23, R7 to R24, R8 to R25, R23 to R26, R45 to R27, R46 to R28, U3 to U10, U8 to U11, U2 to U9
Connections:
- net FB_NODE: now also R66.2, R67.1
- net GNDA: now also R67.2
- net V_IN: now also R66.1

Commit message: [sch] Remote volt-drop detect and NAND latch
Parts:
- removed C34: 10n, Capacitor_SMD:C_0603_1608Metric, symbol Device:C_Small
- removed R25: 1k, Resistor_SMD:R_0603_1608Metric, symbol Device:R_Small
Connections:
- net I_OUT_MON: now also U10.1

Commit message: [layout] change latch -> trigger& software latch (plan)
Parts:
- C21: footprint (none) -> Capacitor_SMD:C_0603_1608Metric
Changed lines of the file:
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@@
 			)
 		)
-		(property "Footprint" ""
+		(property "Footprint" "Capacitor_SMD:C_0603_1608Metric"
 			(at 58.1152 64.77 0)
 			(hide yes)

Commit message: [layout&trace] layout 3 ntc sense.
Need more trace for 3 ntc, need add filter capacitor
Parts:
- added R72, R73: R_Small, Resistor_SMD:R_0603_1608Metric, symbol Device:R_Small
Connections:
- net FB_NODE: now also R72.2, R73.1
- net GNDA: now also R73.2
- net V_OUT: now also R72.1
Other:
- note added: "Add RC for all output"
